File: ErgoDecks/ErgoDecks.kicad_pcb (KiCad board)
At the start: 2 copper layers, 258.4 x 97.8 mm, 70 parts, among them K1 KEYSW, K10 KEYSW, K11 KEYSW, K12 KEYSW, K13 KEYSW, K14 KEYSW, K15 KEYSW, K16 KEYSW, K17 KEYSW, K2 KEYSW, K3 KEYSW, K4 KEYSW, K5 KEYSW, K6 KEYSW, K7 KEYSW, K8 KEYSW, K9 KEYSW, U1 nice_nano

Commit message: Add files via upload
Parts:
- removed the D1 at (269.1, 84.2)
- removed the D10 at (209.3, 71.0)
- removed the D11 at (209.3, 91.2)
- removed the D12 at (209.5, 111.0)
- removed the D13 at (189.6, 74.0)
- removed the D14 at (189.5, 94.0)
- removed the D15 at (189.6, 114.0)
- removed the D16 at (201.2, 133.7)
- removed the D17 at (172.1, 142.8)
- removed the D2 at (269.6, 104.2)
- removed the D3 at (269.5, 124.2)
- removed the D4 at (249.3, 71.0)
- removed the D5 at (249.3, 91.0)
- removed the D6 at (249.3, 111.0)
- removed the D7 at (229.3, 66.0)
- removed the D8 at (229.6, 86.0)
- removed the D9 at (229.6, 106.0)
- removed the K1 at (269.3, 80.0)
- removed the K10 at (209.3, 66.7)
- removed the K11 at (209.3, 86.7)
- removed the K12 at (209.3, 106.7)
- removed the K13 at (189.5, 69.7)
- removed the K14 at (189.5, 89.7)
- removed the K15 at (189.5, 109.7)
- removed the K16 at (200.5, 129.5)
- removed the K17 at (170.3, 139.0)
- removed the K2 at (269.3, 100.0)
- removed the K3 at (269.3, 120.0)
- removed the K4 at (249.3, 66.7)
- removed the K5 at (249.3, 86.7)
- removed the K6 at (249.3, 106.7)
- removed the K7 at (229.3, 61.7)
- removed the K8 at (229.3, 81.7)
- removed the K9 at (229.3, 101.7)
- removed the U1 at (169.0, 70.5)
- K1, K10, K11, K12, K13, K14, K15, K2, K3, K4, K5, K6, K7, K8, K9: footprint keebs.pretty-master:Mx_Alps_100 -> Choc switches:SW_PG1350_reversible
- K16, K17: footprint keebs.pretty-master:Mx_Alps_150 -> Choc switches:SW_PG1350_reversible
- moved D16 17.1 mm to (93.5, 116.8), turned to 170 degrees
- moved D17 16.4 mm to (110.8, 134.2)
- moved D7 15.0 mm to (76.7, 54.2), turned to 180 degrees
- moved D4 14.1 mm to (49.0, 57.0), turned to 180 degrees
- moved D10 13.8 mm to (86.6, 57.0), turned to 180 degrees
- moved D11 13.8 mm to (86.3, 77.2), turned to 180 degrees
- moved D12 13.8 mm to (86.6, 97.2), turned to 180 degrees
- moved D13 13.8 mm to (106.1, 60.2), turned to 180 degrees
- moved D14 13.8 mm to (106.3, 80.2), turned to 180 degrees
- moved D15 13.8 mm to (106.1, 100.2), turned to 180 degrees
- moved D2 13.8 mm to (26.6, 90.5), turned to 180 degrees
- moved D3 13.8 mm to (26.5, 110.5), turned to 180 degrees
- moved D5 13.8 mm to (46.6, 77.2), turned to 180 degrees
- moved D6 13.8 mm to (46.4, 97.2), turned to 180 degrees
- moved D8 13.8 mm to (66.6, 72.2), turned to 180 degrees
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Routing:
- net /Col0: track 344.0 -> 150.0 mm, vias 3 -> 0
- net /Row2: track 289.8 -> 123.1 mm
- net /Row3: track 227.7 -> 71.9 mm
- net /Row1: track 253.4 -> 107.1 mm
- net /Col1: track 281.5 -> 138.9 mm, vias 3 -> 2
- net /Col3: track 245.0 -> 121.9 mm, vias 0 -> 2
- net /Row0: track 218.9 -> 100.6 mm
- net /Col4: track 227.9 -> 110.9 mm
- net /Col2: track 232.0 -> 116.3 mm, vias 0 -> 2
- net Net-(D16-A): track 19.2 -> 29.1 mm
- net Net-(D14-A): track 19.2 -> 28.3 mm, vias 0 -> 3
- net Net-(D4-A): track 19.3 -> 24.7 mm
- net Net-(D10-A): track 19.0 -> 24.3 mm
- net Net-(D6-A): track 19.2 -> 24.0 mm
- net Net-(D5-A): track 19.3 -> 24.1 mm
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Other:
- board size 258.4 x 97.8 mm -> 121.5 x 99.5 mm
