File: ErgoDecks/ErgoDecks.kicad_sch (KiCad schematic)
At the start: 35 parts, among them K1 KEYSW, K10 KEYSW, K11 KEYSW, K12 KEYSW, K13 KEYSW, K14 KEYSW, K15 KEYSW, K16 KEYSW, K17 KEYSW, K2 KEYSW, K3 KEYSW, K4 KEYSW, K5 KEYSW, K6 KEYSW, K7 KEYSW, K8 KEYSW, K9 KEYSW, U1 nice_nano

Commit message: Add files via upload
Parts:
- K1, K10, K11, K12, K13, K14, K15, K2, K3, K4, K5, K6, K7, K8, K9: footprint keebs.pretty-master:Mx_Alps_100 -> Choc switches:SW_PG1350_reversible
- K16, K17: footprint keebs.pretty-master:Mx_Alps_150 -> Choc switches:SW_PG1350_reversible
Changed lines of the file:
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@@
 			)
 		)
-		(property "Footprint" "keebs.pretty-master:Mx_Alps_100"
+		(property "Footprint" "Choc switches:SW_PG1350_reversible"
 			(at 83.82 114.3 0)
 			(effects
@@
 			)
 		)
-		(property "Footprint" "keebs.pretty-master:Mx_Alps_100"
+		(property "Footprint" "Choc switches:SW_PG1350_reversible"
 			(at 101.6 127 0)
 			(effects
@@
 			)
 		)
-		(property "Footprint" "keebs.pretty-master:Mx_Alps_100"
+		(property "Footprint" "Choc switches:SW_PG1350_reversible"
 			(at 101.6 114.3 0)
 			(effects
@@
 			)
 		)
-		(property "Footprint" "keebs.pretty-master:Mx_Alps_100"
+		(property "Footprint" "Choc switches:SW_PG1350_reversible"
 			(at 119.38 139.7 0)
 			(effects
@@
 			)
 		)
-		(property "Footprint" "keebs.pretty-master:Mx_Alps_100"
+		(property "Footprint" "Choc switches:SW_PG1350_reversible"
 			(at 154.94 139.7 0)
 			(effects
@@
 			)
 		)
-		(property "Footprint" "keebs.pretty-master:Mx_Alps_100"
+		(property "Footprint" "Choc switches:SW_PG1350_reversible"
 			(at 83.82 127 0)
 			(effects
@@
 			)
 		)
-		(property "Footprint" "keebs.pretty-master:Mx_Alps_100"
+		(property "Footprint" "Choc switches:SW_PG1350_reversible"
 			(at 137.16 127 0)
 			(effects
@@
 			)
 		)
-		(property "Footprint" "keebs.pretty-master:Mx_Alps_100"
+		(property "Footprint" "Choc switches:SW_PG1350_reversible"
 			(at 101.6 139.7 0)
 			(effects
@@
 			)
 		)
-		(property "Footprint" "keebs.pretty-master:Mx_Alps_100"
+		(property "Footprint" "Choc switches:SW_PG1350_reversible"
 			(at 154.94 114.3 0)
 			(effects
@@
 			)
 		)
-		(property "Footprint" "keebs.pretty-master:Mx_Alps_100"
+		(property "Footprint" "Choc switches:SW_PG1350_reversible"
 			(at 119.38 114.3 0)
 			(effects
@@
 			)
 		)
-		(property "Footprint" "keebs.pretty-master:Mx_Alps_100"
+		(property "Footprint" "Choc switches:SW_PG1350_reversible"
 			(at 154.94 127 0)
 			(effects
@@
 			)
 		)
-		(property "Footprint" "keebs.pretty-master:Mx_Alps_100"
+		(property "Footprint" "Choc switches:SW_PG1350_reversible"
 			(at 83.82 139.7 0)
 			(effects
@@
 			)
 		)
-		(property "Footprint" "keebs.pretty-master:Mx_Alps_150"
+		(property "Footprint" "Choc switches:SW_PG1350_reversible"
 			(at 154.94 152.4 0)
 			(effects
@@
 			)
 		)
-		(property "Footprint" "keebs.pretty-master:Mx_Alps_100"
+		(property "Footprint" "Choc switches:SW_PG1350_reversible"
 			(at 119.38 127 0)
 			(effects
@@
 			)
 		)
-		(property "Footprint" "keebs.pretty-master:Mx_Alps_150"
+		(property "Footprint" "Choc switches:SW_PG1350_reversible"
 			(at 137.16 152.4 0)
 			(effects
@@
 			)
 		)
-		(property "Footprint" "keebs.pretty-master:Mx_Alps_100"
+		(property "Footprint" "Choc switches:SW_PG1350_reversible"
 			(at 137.16 114.3 0)
 			(effects
@@
 			)
 		)
-		(property "Footprint" "keebs.pretty-master:Mx_Alps_100"
+		(property "Footprint" "Choc switches:SW_PG1350_reversible"
 			(at 137.16 139.7 0)
 			(effects
